File: Alpenglow_SunnySurprise_PCB.kicad_sch (KiCad schematic)
At the start: 7 parts, among them SW1 SW_SPDT

Commit message: Updated switch footprint
Parts:
- SW1: footprint Alpenglow:SW_SLIDE_RTA -> Alpenglow:SW_SPDT_SLIDE_THRU_RTA
Changed lines of the file:
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@@
     (property "Reference" "SW1" (id 0) (at 133.35 58.801 0))
     (property "Value" "SW_SPDT" (id 1) (at 133.35 61.1124 0))
-    (property "Footprint" "Alpenglow:SW_SLIDE_RTA" (id 2) (at 133.35 66.04 0)
+    (property "Footprint" "Alpenglow:SW_SPDT_SLIDE_THRU_RTA" (id 2) (at 133.35 66.04 0)
       (effects (font (size 1.27 1.27)) hide)
     )
@@
     )
     (path "/00000000-0000-0000-0000-0000622bdc31"
-      (reference "SW1") (unit 1) (value "SW_SPDT") (footprint "Alpenglow:SW_SLIDE_RTA")
+      (reference "SW1") (unit 1) (value "SW_SPDT") (footprint "Alpenglow:SW_SPDT_SLIDE_THRU_RTA")
     )
   )

Commit message: Updated Switch, Removed GND pour and added GND traces, Updated artwork
Parts:
- SW1: footprint Alpenglow:SW_SPDT_SLIDE_THRU_RTA -> Alpenglow:Alpenglow_SW_SPDT_3pin_RTA
Changed lines of the file:
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@@
     (property "Reference" "SW1" (id 0) (at 133.35 58.801 0))
     (property "Value" "SW_SPDT" (id 1) (at 133.35 61.1124 0))
-    (property "Footprint" "Alpenglow:SW_SPDT_SLIDE_THRU_RTA" (id 2) (at 133.35 66.04 0)
+    (property "Footprint" "Alpenglow:Alpenglow_SW_SPDT_3pin_RTA" (id 2) (at 133.35 66.04 0)
       (effects (font (size 1.27 1.27)) hide)
     )
@@
     )
     (path "/00000000-0000-0000-0000-0000622bdc31"
-      (reference "SW1") (unit 1) (value "SW_SPDT") (footprint "Alpenglow:SW_SPDT_SLIDE_THRU_RTA")
+      (reference "SW1") (unit 1) (value "SW_SPDT") (footprint "Alpenglow:Alpenglow_SW_SPDT_3pin_RTA")
     )
   )

Commit message: Updated font, Removed extra vias for GND traces, Renamed pwr net to LED+
Connections:
- net LED+: now reaches D1.2 (A), D2.2 (A), D3.2 (A), D4.2 (A), D5.2 (A), SW1.3 (C)
Changed lines of the file:
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@@
     (stroke (width 0) (type default) (color 0 0 0 0))
+  )
+  (label "LED+" (at 165.1 68.58 0)
+    (effects (font (size 1.27 1.27)) (justify left bottom))
   )
   (symbol (lib_id "Device:Battery_Cell") (at 78.74 90.17 0) (unit 1)
